File: capsule.kicad_sch (KiCad schematic)
At the start: 90 parts, among them J1 OLED-128x64, J2 Conn_01x01_Socket, SW1 SW, SW10 SW, SW11 SW, SW12 SW, SW13 SW, SW14 SW, SW15 SW, SW16 SW, SW17 SW, SW18 SW, SW19 SW, SW2 SW, SW20 SW, SW21 SW, SW22 SW, SW23 SW, SW24 SW, SW25 SW, SW26 SW, SW27 SW, SW28 SW, SW29 SW, SW3 SW, SW30 SW, SW31 SW, SW32 SW, SW33 SW, SW34 SW, SW35 SW, SW36 SW, SW4 SW, SW5 SW, SW6 SW, SW7 SW, SW8 SW, SW9 SW, U1 ProMicro

Commit message: SCH refactor
Parts:
- removed D16, D17, D18, D34, D35, D36: D, 0-jasonhazel-footprints:D_SOD-123_via, symbol hazel:D
- removed SW16, SW17, SW18, SW34, SW35, SW36: SW, 0-jasonhazel-footprints:jh-choc, symbol hazel:SW
- J1: value OLED-128x64 -> OLED-128x128
- renumbered D19 to D16, D20 to D17, D21 to D18, D22 to D19, D23 to D20, D24 to D21, D25 to D22, D26 to D23, D27 to D24, D28 to D25, D29 to D26, D30 to D27, D31 to D28, D32 to D29, D33 to D30, SW19 to SW16, SW20 to SW17, SW21 to SW18, SW22 to SW19, SW23 to SW20, SW24 to SW21, SW25 to SW22, SW26 to SW23, SW27 to SW24, SW28 to SW25, SW29 to SW26, SW30 to SW27, SW31 to SW28, SW32 to SW29, SW33 to SW30

Commit message: add submodules
Parts:
- D1, D10, D11, D12, D13, D14, D15, D16, D17, D18, D19, D2, D20, D21, D22, D23, D24, D25, D26, D27, D28, D29, D3, D30, D4, D5, D6, D7, D8, D9: footprint 0-jasonhazel-footprints:D_SOD-123_via -> Diode_SMD:D_SOD-123
- H1, H10, H11, H12, H2, H3, H4, H5, H6, H7, H8, H9: footprint 0-jasonhazel-footprints:MountingHole_3.2mm_M3_thinpad -> MountingHole:MountingHole_3.2mm_M3_Pad_Via
- PWR1: footprint 0-jasonhazel-footprints:SPDT_C128955 -> Button_Switch_SMD:SW_SPDT_PCM12
- RESET1: footprint 0-jasonhazel-footprints:SW_SPST_TL3342 -> Button_Switch_SMD:SW_SPST_TL3342
- SW1, SW10, SW11, SW12, SW13, SW14, SW15, SW16, SW17, SW18, SW19, SW2, SW20, SW21, SW22, SW23, SW24, SW25, SW26, SW27, SW28, SW29, SW3, SW30, SW4, SW5, SW6, SW7, SW8, SW9: footprint 0-jasonhazel-footprints:jh-choc -> Kailh_Choc:KailhChoc-1U

Commit message: sch refactor
Parts:
- U1: footprint 0-jasonhazel-footprints:ArduinoProMicro -> Keebio-Parts:ArduinoProMicro
Changed lines of the file:
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@@
       (effects (font (size 1.524 1.524)))
     )
-    (property "Footprint" "0-jasonhazel-footprints:ArduinoProMicro" (at 58.42 97.79 90)
+    (property "Footprint" "Keebio-Parts:ArduinoProMicro" (at 58.42 97.79 90)
       (effects (font (size 1.524 1.524)) hide)
     )
