File: capsule.kicad_sch (KiCad schematic)
At the start: 78 parts, among them J1 OLED-128x128, J2 Conn_01x01_Socket, SW1 SW, SW10 SW, SW11 SW, SW12 SW, SW13 SW, SW14 SW, SW15 SW, SW16 SW, SW17 SW, SW18 SW, SW19 SW, SW2 SW, SW20 SW, SW21 SW, SW22 SW, SW23 SW, SW24 SW, SW25 SW, SW26 SW, SW27 SW, SW28 SW, SW29 SW, SW3 SW, SW30 SW, SW4 SW, SW5 SW, SW6 SW, SW7 SW, SW8 SW, SW9 SW, U1 ProMicro

Commit message: sch refactor
Parts:
- removed U1: ProMicro, Keebio-Parts:ArduinoProMicro, symbol keebio:ProMicro
- added C1: 1uF, symbol Device:C_Small
- added C2, C3, C4, C5: 0.1uF, symbol Device:C_Small
- added C6: 10uF, symbol Device:C_Small
- added C7, C8: 22pF, symbol Device:C_Small
- added R1, R4: 10k, symbol Device:R_Small
- added R2, R3: 22, symbol Device:R_Small
- added SW31: SW_Push, symbol Switch:SW_Push
- added U2: ATmega32U4-A, Package_QFP:TQFP-44_10x10mm_P0.8mm, symbol MCU_Microchip_ATmega:ATmega32U4-A
- added Y1: 16MHz, symbol Device:Crystal_GND24_Small
Connections:
- net GND: now also C1.2, C2.2, C3.2, C4.2, C5.2, C6.2, C7.2, C8.2, R1.2, SW31.1, U2.15 (GND), U2.23 (GND), U2.35 (GND), U2.43 (GND), U2.5 (UGND), Y1.2, Y1.4
- new net: R1.1, U2.33 (~{HWB}/PE2)
- new net: C7.1, U2.17 (XTAL1), Y1.1
- new net: C8.1, U2.16 (XTAL2), Y1.3
- new net: R2.2, U2.4 (D+)
- new net: R4.2, SW31.2, U2.13 (~{RESET})
- new net: R3.2, U2.3 (D-)
- new net: C1.1, U2.6 (UCAP)
- new net +5V: C2.1, C3.1, C4.1, C5.1, C6.1, R4.1, U2.14 (VCC), U2.2 (UVCC), U2.24 (AVCC), U2.34 (VCC), U2.44 (AVCC), U2.7 (VBUS)
- new net D+: R2.1
- new net D-: R3.1
Other:
- moved on the sheet: BT1, D1, D10, D11, D12, D13, D14, D15, D16, D17, D18, D19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

Commit message: sch refactor
Parts:
- removed BT1: Battery, 0-jasonhazel-footprints:3JST_BAT, symbol Device:Battery
- removed J1: OLED-128x128, 0-jasonhazel-footprints:OLED-128x64, symbol display:OLED-128x64
- removed PWR1: SW_SPDT, Button_Switch_SMD:SW_SPDT_PCM12, symbol Switch:SW_SPDT
- removed RESET1: SW, Button_Switch_SMD:SW_SPST_TL3342, symbol hazel:SW
- added F1: 500mA, symbol Device:Polyfuse_Small
- added USB1: Molex-0548190589, symbol random-keyboard-parts:Molex-0548190589
- renumbered D3 to D1, D18 to D10, D6 to D2, D9 to D3, D12 to D4, D15 to D5, D30 to D6, D27 to D7, D24 to D8, D21 to D9, SW18 to SW10, SW6 to SW2, SW9 to SW3, SW12 to SW4, SW15 to SW5, SW30 to SW6, SW27 to SW7, SW24 to SW8, SW21 to SW9
Connections:
- net +5V: now also F1.2
- net D+: now also USB1.3 (D+)
- net D-: now also USB1.4 (D-)
- net GND: now also USB1.1 (GND)
- net row0 renamed ROW0
- net row1 renamed ROW1
- net row2 renamed ROW2
- new net: F1.1, USB1.5 (VBUS)

Commit message: sch refactor
Parts:
- removed J2: Conn_01x01_Socket, 0-jasonhazel-footprints:CS_PIN, symbol Connector:Conn_01x01_Socket
- C1, C2, C3, C4, C5, C6, C7, C8: footprint (none) -> Capacitor_SMD:C_0805_2012Metric
- F1: footprint (none) -> Fuse:Fuse_1206_3216Metric
- R1, R2, R3, R4: footprint (none) -> Resistor_SMD:R_0805_2012Metric
- SW31: footprint (none) -> random-keyboard-parts:SKQG-1155865
- USB1: footprint (none) -> random-keyboard-parts:Molex-0548190589
- Y1: footprint (none) -> Crystal:Crystal_SMD_3225-4Pin_3.2x2.5mm
- renumbered D2 to D11, D5 to D12, D8 to D13, D11 to D14, D14 to D15, D29 to D16, D26 to D17, D23 to D18, D20 to D19, D17 to D20, D1 to D21, D4 to D22, D7 to D23, D10 to D24, D13 to D25, D28 to D26, D25 to D27, D22 to D28, D19 to D29, D16 to D30, SW2 to SW11, SW5 to SW12, SW8 to SW13, SW11 to SW14, SW14 to SW15, SW29 to SW16, SW26 to SW17, SW23 to SW18, SW20 to SW19, SW17 to SW20, SW3 to SW21, SW4 to SW22, SW7 to SW23, SW10 to SW24, SW13 to SW25, SW28 to SW26, SW25 to SW27, SW22 to SW28, SW19 to SW29, SW16 to SW30
Connections:
- net row4 is gone; now on net ROW0: D10.1, D6.1, D7.1, D8.1, D9.1
- net row5 is gone; now on net ROW1: D16.1, D17.1, D18.1, D19.1, D20.1
- net row6 is gone; now on net ROW2: D26.1, D27.1, D28.1, D29.1, D30.1
- net col0 renamed COL0
- net COL0: no longer SW10.2, SW20.2, SW30.2
- net col1 renamed COL1
- net COL1: no longer SW19.2, SW29.2, SW9.2
- net col2 renamed COL2
- net COL2: no longer SW18.2, SW28.2, SW8.2
- net col3 renamed COL3
- net COL3: no longer SW17.2, SW27.2, SW7.2
- net col4 renamed COL4
- net COL4: no longer SW16.2, SW26.2, SW6.2
- new net COL5: SW16.2, SW26.2, SW6.2
- new net COL6: SW17.2, SW27.2, SW7.2
- new net COL7: SW18.2, SW28.2, SW8.2
- new net COL8: SW19.2, SW29.2, SW9.2
- new net COL9: SW10.2, SW20.2, SW30.2

Commit message: pcb refactor
Parts:
- removed C1: 1uF, Capacitor_SMD:C_0805_2012Metric, symbol Device:C_Small
- removed C2, C3, C4, C5: 0.1uF, Capacitor_SMD:C_0805_2012Metric, symbol Device:C_Small
- removed C6: 10uF, Capacitor_SMD:C_0805_2012Metric, symbol Device:C_Small
- removed C7, C8: 22pF, Capacitor_SMD:C_0805_2012Metric, symbol Device:C_Small
- removed F1: 500mA, Fuse:Fuse_1206_3216Metric, symbol Device:Polyfuse_Small
- removed H1, H10, H11, H12, H2, H3, H4, H5, H6, H7, H8, H9: MountingHole, MountingHole:MountingHole_3.2mm_M3_Pad_Via, symbol Mechanical:MountingHole
- removed R1, R4: 10k, Resistor_SMD:R_0805_2012Metric, symbol Device:R_Small
- removed R2, R3: 22, Resistor_SMD:R_0805_2012Metric, symbol Device:R_Small
- removed U2: ATmega32U4-A, Package_QFP:TQFP-44_10x10mm_P0.8mm, symbol MCU_Microchip_ATmega:ATmega32U4-A
- removed USB1: Molex-0548190589, random-keyboard-parts:Molex-0548190589, symbol random-keyboard-parts:Molex-0548190589
- removed Y1: 16MHz, Crystal:Crystal_SMD_3225-4Pin_3.2x2.5mm, symbol Device:Crystal_GND24_Small
- added U1: rp2040-zero, mcu:rp2040-zero-tht, symbol mcu:rp2040-zero
- SW1, SW10, SW11, SW12, SW13, SW14, SW15, SW16, SW17, SW18, SW19, SW2, SW20, SW21, SW22, SW23, SW24, SW25, SW26, SW27, SW28, SW29, SW3, SW30, SW4, SW5, SW6, SW7, SW8, SW9: footprint Kailh_Choc:KailhChoc-1U -> miketronic_fplib:MB_KailhChoc-1U
Connections:
- net GND: no longer names the net of SW31.1

Commit message: add submodules
Parts:
- removed SW31: SW_Push, random-keyboard-parts:SKQG-1155865, symbol Switch:SW_Push
- added Connector1: MB_i2c_header, miketronic_fplib:MB_I2C_Breakout_reverse, symbol MB_i2c_header:MB_i2c_header
- added LED01, LED02: WS2812B, LED_SMD:LED_WS2812B_PLCC4_5.0x5.0mm_P3.2mm, symbol LED:WS2812B
- D1, D10, D11, D12, D13, D14, D15, D16, D17, D18, D19, D2, D20, D21, D22, D23, D24, D25, D26, D27, D28, D29, D3, D30, D4, D5, D6, D7, D8, D9: footprint Diode_SMD:D_SOD-123 -> miketronic_fplib:MB_D_SOD-123_1PAD
- SW1, SW10, SW11, SW12, SW13, SW14, SW15, SW16, SW17, SW18, SW19, SW2, SW20, SW21, SW22, SW23, SW24, SW25, SW26, SW27, SW28, SW29, SW3, SW30, SW4, SW5, SW6, SW7, SW8, SW9: footprint miketronic_fplib:MB_KailhChoc-1U -> miketronic_fplib:MB_KailhChoc-1U_17mm
- U1: footprint mcu:rp2040-zero-tht -> miketronic_fplib:MB_rp2040-zero-tht
Connections:
- net COL0: now also U1.4 (3)
- net COL1: now also U1.5 (4)
- net COL2: now also U1.6 (5)
- net COL3: now also U1.7 (6)
- net COL4: now also U1.8 (7)
- net COL5: now also U1.14 (13)
- net COL6: now also U1.15 (14)
- net COL7: now also U1.17 (26)
- net COL8: now also U1.18 (27)
- net COL9: now also U1.19 (28)
- net ROW0: now also U1.1 (0); no longer D10.1, D6.1, D7.1, D8.1, D9.1
- net ROW1: now also U1.2 (1); no longer D16.1, D17.1, D18.1, D19.1, D20.1
- net ROW2: now also U1.3 (2); no longer D26.1, D27.1, D28.1, D29.1, D30.1
- net RGB: now reaches U1.10 (9)
- net RGB: now also LED01.4 (DIN)
- net SDA: now reaches U1.11 (10)
- net SDA: now also Connector1.4 (SDA)
- net SCL: now reaches U1.12 (11)
- net SCL: now also Connector1.3 (SCL)
- net ROW5: now reaches U1.13 (12)
- net ROW5: now also D26.1, D27.1, D28.1, D29.1, D30.1
- net ROW4: now reaches U1.16 (15)
- net ROW4: now also D16.1, D17.1, D18.1, D19.1, D20.1
- net ROW3: now reaches U1.20 (29)
- net ROW3: now also D10.1, D6.1, D7.1, D8.1, D9.1
- net GND: now reaches U1.22 (GND)
- net GND: now also Connector1.1 (GND), LED01.3 (VSS), LED02.3 (VSS)
- net VCC: now reaches U1.23 (5V)
- net VCC: now also Connector1.5 (VCC), LED01.1 (VDD), LED02.1 (VDD)
- new net: LED01.2 (DOUT), LED02.4 (DIN)
- no-connect marks 0 -> 2
