File: Capsule - INTMCU.kicad_pcb (KiCad board)
At the start: 2 copper layers, 239 x 67.4 mm, 90 parts, among them J1 USB_C_Receptacle, SW1 SW, SW10 SW, SW11 SW, SW12 SW, SW13 SW, SW14 SW, SW15 SW, SW16 SW, SW17 SW, SW18 SW, SW19 SW, SW2 SW, SW20 SW, SW21 SW, SW22 SW, SW23 SW, SW24 SW, SW25 SW, SW26 SW, SW27 SW, SW28 SW, SW29 SW, SW3 SW, SW30 SW, SW31 SW_Push, SW4 SW, SW5 SW, SW6 SW, SW7 SW, SW8 SW, SW9 SW, U2 ATmega32U4-A, U3 TPD2S017, Y1 16MHz

Commit message: big update
Parts:
- removed H1, H10, H11, H12, H2, H3, H4, H5, H6, H7, H8, H9: MountingHole, MountingHole:MountingHole_3.2mm_M3_Pad_Via
- removed J1: USB_C_Receptacle, Connector_USB:USB_C_Receptacle_XKB_U262-16XN-4BVC11
- removed the R2 at (137.2, 33.0)
- removed R3: 22, Resistor_SMD:R_0805_2012Metric
- removed U3: TPD2S017, Package_TO_SOT_SMD:SOT-23-6
- removed Y1: 16MHz, Crystal:Crystal_SMD_3225-4Pin_3.2x2.5mm
- added C9: 4.7uF, Capacitor_SMD:C_0805_2012Metric, B.Cu at (124.2, 27.4)
- added U2: PRTR5V0U2X, Keebio-Parts:SOT-143B, B.Cu at (138.0, 36.5)
- added UR1: 1M, Keebio-Parts:R_0805, B.Cu at (129.4, 27.5)
- added UR2: 5.1k, Keebio-Parts:R_0805, B.Cu at (134.0, 31.5)
- added UR3: 5.1k, Keebio-Parts:R_0805, B.Cu at (143.0, 32.0)
- added UR4: 22, Keebio-Parts:R_0805, B.Cu at (136.8, 41.3)
- added UR5: 22, Keebio-Parts:R_0805, B.Cu at (139.3, 41.3)
- added USB1: HRO-TYPE-C-31-M-12, Keebio-Parts:HRO-TYPE-C-31-M-12-Assembly, B.Cu at (138.5, 19.4)
- added X1: XTAL_GND, Crystal:Crystal_SMD_3225-4Pin_3.2x2.5mm, B.Cu at (149.3, 64.8)
- C1: renamed from C7; moved to B.Cu
- C2: renamed from C8; moved to B.Cu
- C3: renamed from C2; moved to B.Cu
- C4: renamed from C3; moved to B.Cu
- C5: renamed from C4; moved to B.Cu
- C6: renamed from C5; moved to B.Cu
- C7: renamed from C6; moved to B.Cu
- C8: renamed from C1; value 4.7uF -> 1uF; moved to B.Cu
- D1, D10, D11, D12, D13, D14, D15, D16, D17, D18, D19, D2, D20, D21, D22, D23, D24, D25, D26, D27, D28, D29, D3, D30, D4, D5, D6, D7, D8, D9: footprint Diode_SMD:D_SOD-123 -> miketronic_fplib:Diode-Hybrid-Back; moved to F.Cu
- F1: value 500mA -> 500mA Hold; moved to B.Cu
- R1: renamed from R4; moved to B.Cu
- R2: renamed from R1; moved to B.Cu
- SW1, SW10, SW11, SW12, SW13, SW14, SW15, SW16, SW17, SW18, SW19, SW2, SW20, SW21, SW22, SW23, SW24, SW25, SW26, SW27, SW28, SW29, SW3, SW30, SW4, SW5, SW6, SW7, SW8, SW9: footprint marbastlib-choc:SW_choc_v1_1u -> miketronic_fplib:MB_KailhChoc-1U_17mm
- SW50: renamed from SW31; moved to B.Cu
- U1: renamed from U2; value ATmega32U4-A -> ATmega32U4; moved to B.Cu
- moved D1 95.5 mm to (93.6, 115.2), turned to 90 degrees
- moved D11 89.5 mm to (93.6, 125.9), turned to 90 degrees
- moved D21 84.5 mm to (93.6, 136.7), turned to 90 degrees
- moved D2 83.3 mm to (91.6, 115.2), turned to 90 degrees
- moved D10 81.3 mm to (171.6, 86.2), turned to 90 degrees
- moved D20 77.2 mm to (171.6, 96.8), turned to 90 degrees
- moved D12 76.2 mm to (91.6, 125.9), turned to 90 degrees
- moved D5 75.3 mm to (85.6, 115.2), turned to 90 degrees
- moved D3 75.0 mm to (89.6, 115.2), turned to 90 degrees
- moved D30 73.0 mm to (171.6, 107.4), turned to 90 degrees
- moved D4 72.2 mm to (87.6, 115.2), turned to 90 degrees
- moved D22 70.2 mm to (91.6, 136.7), turned to 90 degrees
- moved D15 67.4 mm to (85.6, 125.9), turned to 90 degrees
- moved D13 67.1 mm to (89.6, 125.9), turned to 90 degrees
- moved D9 64.5 mm to (173.6, 86.2), turned to 90 degrees
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Connections:
- net Net-(U2-XTAL2) renamed XTAL1
- C1 pad 1: Net-(U2-XTAL1) -> GND
- C1 pad 2: GND -> XTAL2
- C3 pad 1: +5V -> VCC
- C4 pad 1: +5V -> VCC
- C5 pad 1: +5V -> VCC
- C6 pad 1: +5V -> VCC
- C7 pad 1: +5V -> VCC
- C8 pad 1: Net-(U2-UCAP) -> GND
- C8 pad 2: GND -> Net-(U1-UCap)
- D10 pad 1: ROW0 -> ROW3
- D16 pad 1: ROW1 -> ROW4
- D17 pad 1: ROW1 -> ROW4
- D18 pad 1: ROW1 -> ROW4
- D19 pad 1: ROW1 -> ROW4
- D20 pad 1: ROW1 -> ROW4
- D26 pad 1: ROW2 -> ROW5
- D27 pad 1: ROW2 -> ROW5
- D28 pad 1: ROW2 -> ROW5
- D29 pad 1: ROW2 -> ROW5
- D30 pad 1: ROW2 -> ROW5
- D6 pad 1: ROW0 -> ROW3
- D7 pad 1: ROW0 -> ROW3
- D8 pad 1: ROW0 -> ROW3
- D9 pad 1: ROW0 -> ROW3
- F1 pad 1: Net-(USB1-VBUS) -> VCC
- R1 pad 1: +5V -> VCC
- U1 pad 14: +5V -> VCC
- U1 pad 17: Net-(U2-XTAL1) -> XTAL2
- U1 pad 18: unconnected-(U2-PD0-Pad18) -> COL5
- U1 pad 19: unconnected-(U2-PD1-Pad19) -> COL6
- U1 pad 2: +5V -> VCC
- U1 pad 20: unconnected-(U2-PD2-Pad20) -> COL7
- U1 pad 21: unconnected-(U2-PD3-Pad21) -> COL8
- U1 pad 22: unconnected-(U2-PD5-Pad22) -> COL9
- U1 pad 24: +5V -> VCC
- U1 pad 28: unconnected-(U2-PB4-Pad28) -> COL0
- U1 pad 29: unconnected-(U2-PB5-Pad29) -> COL1
- U1 pad 3: Net-(U2-D-) -> D-
- U1 pad 30: unconnected-(U2-PB6-Pad30) -> COL2
- U1 pad 31: unconnected-(U2-PC6-Pad31) -> COL3
- U1 pad 32: unconnected-(U2-PC7-Pad32) -> COL4
- U1 pad 34: +5V -> VCC
- U1 pad 36: unconnected-(U2-PF7-Pad36) -> ROW5
- U1 pad 37: unconnected-(U2-PF6-Pad37) -> ROW4
- U1 pad 38: unconnected-(U2-PF5-Pad38) -> ROW3
- U1 pad 39: unconnected-(U2-PF4-Pad39) -> ROW2
- U1 pad 4: Net-(U2-D+) -> D+
- U1 pad 40: unconnected-(U2-PF1-Pad40) -> ROW1
- U1 pad 41: unconnected-(U2-PF0-Pad41) -> ROW0
- U1 pad 44: +5V -> VCC
- U1 pad 6: Net-(U2-UCAP) -> Net-(U1-UCap)
- U1 pad 7: +5V -> VCC
Routing:
- net VCC: track 0.00 -> 165.6 mm, vias 0 -> 10
- net GND: track 0.00 -> 127.5 mm, vias 0 -> 4
- net Net-(U1-~{RESET}): track 0.00 -> 76.2 mm
- net Net-(USB1-SHIELD): track 0.00 -> 37.5 mm
- net XTAL2: track 0.00 -> 23.3 mm
- net Net-(U2-IO1): track 0.00 -> 18.0 mm
- net D+: track 0.00 -> 17.5 mm
- net Net-(U2-IO2): track 0.00 -> 16.8 mm
- net D-: track 0.00 -> 16.8 mm
- net +5V: track 9.60 -> 0.00 mm
- net XTAL1: track 0.00 -> 9.38 mm
- net Net-(USB1-CC2): track 0.00 -> 5.64 mm
- net Net-(USB1-CC1): track 0.00 -> 5.32 mm
- net Net-(U1-UCap): track 0.00 -> 4.19 mm
- net Net-(U1-~{HWB/PE2}): track 0.00 -> 3.32 mm
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- added copper zone on B.Cu, net GND
- added copper zone on F.Cu, net GND
Other:
- board outline removed
