File: capsule - INTMCU.kicad_sch (KiCad schematic)
At the start: 91 parts, among them J1 USB_C_Receptacle, SW1 SW, SW10 SW, SW11 SW, SW12 SW, SW13 SW, SW14 SW, SW15 SW, SW16 SW, SW17 SW, SW18 SW, SW19 SW, SW2 SW, SW20 SW, SW21 SW, SW22 SW, SW23 SW, SW24 SW, SW25 SW, SW26 SW, SW27 SW, SW28 SW, SW29 SW, SW3 SW, SW30 SW, SW31 SW_Push, SW4 SW, SW5 SW, SW6 SW, SW7 SW, SW8 SW, SW9 SW, U2 ATmega32U4-A, U3 TPD2S017, Y1 16MHz

Commit message: big update
Parts:
- removed F1: 500mA, Fuse:Fuse_1206_3216Metric, symbol Device:Polyfuse_Small
- removed H1, H10, H11, H12, H2, H3, H4, H5, H6, H7, H8, H9: MountingHole, MountingHole:MountingHole_3.2mm_M3_Pad_Via, symbol Mechanical:MountingHole
- removed J1: USB_C_Receptacle, Connector_USB:USB_C_Receptacle_XKB_U262-16XN-4BVC11, symbol Connector:USB_C_Receptacle
- removed R2, R3: 22, Resistor_SMD:R_0805_2012Metric, symbol Device:R_Small
- removed U3: TPD2S017, Package_TO_SOT_SMD:SOT-23-6, symbol Power_Protection:TPD2S017
- removed USB1: USB_C_Receptacle_XKB_U262-16XN-4BVC11, Connector_USB:USB_C_Receptacle_XKB_U262-16XN-4BVC11, symbol random-keyboard-parts:Molex-0548190589
- removed Y1: 16MHz, Crystal:Crystal_SMD_3225-4Pin_3.2x2.5mm, symbol Device:Crystal_GND24_Small
- added C9: 4.7uF, Capacitor_SMD:C_0805_2012Metric, symbol cpm43-rescue:C_Small-device
- added F1: 500mA Hold, Fuse:Fuse_1206_3216Metric, symbol cpm43-rescue:Polyfuse_Small-device
- added U2: PRTR5V0U2X, Keebio-Parts:SOT-143B, symbol ai03-locallib:PRTR5V0U2X
- added UR1: 1M, Keebio-Parts:R_0805, symbol cpm43-rescue:R-device
- added UR2, UR3: 5.1k, Keebio-Parts:R_0805, symbol cpm43-rescue:R-device
- added UR4, UR5: 22, Keebio-Parts:R_0805, symbol cpm43-rescue:R-device
- added USB1: HRO-TYPE-C-31-M-12, Keebio-Parts:HRO-TYPE-C-31-M-12-Assembly, symbol Type-C:HRO-TYPE-C-31-M-12
- added X1: XTAL_GND, Crystal:Crystal_SMD_3225-4Pin_3.2x2.5mm, symbol keyboard_parts:XTAL_GND
- D1, D10, D11, D12, D13, D14, D15, D16, D17, D18, D19, D2, D20, D21, D22, D23, D24, D25, D26, D27, D28, D29, D3, D30, D4, D5, D6, D7, D8, D9: footprint Diode_SMD:D_SOD-123 -> miketronic_fplib:Diode-Hybrid-Back
- SW1, SW10, SW11, SW12, SW13, SW14, SW15, SW16, SW17, SW18, SW19, SW2, SW20, SW21, SW22, SW23, SW24, SW25, SW26, SW27, SW28, SW29, SW3, SW30, SW4, SW5, SW6, SW7, SW8, SW9: footprint marbastlib-choc:SW_choc_v1_1u -> miketronic_fplib:MB_KailhChoc-1U_17mm
- U1: renamed from U2; value ATmega32U4-A -> ATmega32U4; symbol MCU_Microchip_ATmega:ATmega32U4-A -> keyboard_parts:ATMEGA32U4
- renumbered C7 to C1, C8 to C2, C2 to C3, C3 to C4, C4 to C5, C5 to C6, C6 to C7, C1 to C8, R4 to R1, R1 to R2, SW31 to SW50
Connections:
- net +5V: now also F1.2; no longer C3.1, C4.1, C5.1, C6.1, C7.1, R1.1, U1.14 (VCC), U1.2 (UVCC), U1.24 (AVCC), U1.34 (VCC), U1.44 (AVCC), U1.7 (VBUS)
- net COL0: now also U1.28 (PB4)
- net COL1: now also U1.29 (PB5)
- net COL2: now also U1.30 (PB6)
- net COL3: now also U1.31 (PC6)
- net COL4: now also U1.32 (PC7)
- net COL5: now also U1.18 (PD0/INT0)
- net COL6: now also U1.19 (PD1/INT1)
- net COL7: now also U1.20 (PD2/RXD1)
- net COL8: now also U1.21 (PD3/TXD1)
- net COL9: now also U1.22 (PD5/XCK1)
- net D+: now also U1.4 (D+), UR5.1
- net D-: now also U1.3 (D-), UR4.2
- net GND: now also C1.1, C8.1, C9.1, U2.1 (GND), UR1.1, UR2.2, UR3.1, USB1.1 (GND), USB1.12 (GND), X1.3; no longer C1.2, C8.2
- net ROW0: now also U1.41 (PF0); no longer D10.1, D6.1, D7.1, D8.1, D9.1
- net ROW1: now also U1.40 (PF1); no longer D16.1, D17.1, D18.1, D19.1, D20.1
- net ROW2: now also U1.39 (PF4); no longer D26.1, D27.1, D28.1, D29.1, D30.1
- net XTAL2: now reaches U1.17 (XTAL2)
- net XTAL2: now also C1.2, X1.1; no longer C1.1
- net XTAL1: now reaches C2.1, U1.16 (XTAL1)
- net XTAL1: now also X1.2
- net at U1.6 (UCap): now also C8.2; no longer C8.1
- net ROW5: now reaches U1.36 (PF7)
- net ROW5: now also D26.1, D27.1, D28.1, D29.1, D30.1
- net ROW4: now reaches U1.37 (PF6)
- net ROW4: now also D16.1, D17.1, D18.1, D19.1, D20.1
- net ROW3: now reaches U1.38 (PF5)
- net ROW3: now also D10.1, D6.1, D7.1, D8.1, D9.1
- new net: U2.2 (IO1), UR5.2, USB1.6 (DP1), USB1.8 (DP2)
- new net: U2.3 (IO2), UR4.1, USB1.5 (DN2), USB1.7 (DN1)
- new net: C9.2, UR1.2, USB1.13 (SHIELD)
- new net: UR3.2, USB1.10 (CC2)
- new net: UR2.1, USB1.4 (CC1)
- new net VCC: C3.1, C4.1, C5.1, C6.1, C7.1, F1.1, R1.1, U1.14 (VCC), U1.2 (UVcc), U1.24 (AVCC), U1.34 (VCC), U1.44 (AVCC), U1.7 (VBus), U2.4 (VCC), USB1.11 (VBUS), USB1.2 (VBUS)
- no-connect marks 0 -> 12
Other:
- moved on the sheet: C1, C2, C3, C4, C5, C6, C7, C8, D1, D10, D11, D12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
